File: KiCad/VWS-SDR-ref-design.kicad_sch (KiCad schematic)
At the start: 99 parts, among them J1 RF_IN, J10 IF breakout, J2 IQ_Out, J3 SI5351 board, J4 Conn_01x20_Socket, J5 Conn_01x20_Socket, J6 I2C breakout, J7 Power breakout, J8 GPIO Breakout, J9 GPIO Breakout, U1 GALI-S66, U2 74CBTLV3253DR, U3 MC33078, U4 MC33078, U5 RASPBERRY-PICO

Commit message: Placement complete, next step routing
Parts:
- removed J8: GPIO Breakout, symbol Connector:Conn_01x14_Pin
- added G10, G9: TestPoint, Connector_PinHeader_2.54mm:PinHeader_1x01_P2.54mm_Vertical, symbol Connector:TestPoint
- added J8: GPIO Breakout, Connector_PinSocket_2.54mm:PinSocket_1x15_P2.54mm_Vertical, symbol Connector:Conn_01x15_Pin
- C1, C10, C11, C12, C13, C14, C15, C16, C17, C18, C19, C2, C20, C21, C22, C23, C24, C26, C27, C29, C3, C30, C4, C5, C6, C7, C8, C9: footprint Capacitor_SMD:C_1206_3216Metric -> Capacitor_SMD:C_1206_3216Metric_Pad1.33x1.80mm_HandSolder
- J1: footprint Connector_Coaxial:SMA_Amphenol_901-144_Vertical -> VWS-SDR:SMA_Vertical_and_Edgemount
- J10: footprint (none) -> Connector_PinSocket_2.54mm:PinSocket_1x03_P2.54mm_Vertical
- J9: footprint (none) -> Connector_PinSocket_2.54mm:PinSocket_1x10_P2.54mm_Vertical
- L1, L2, L3, L4, L5, L6, R1, R10, R11, R12, R13, R14, R15, R16, R17, R18, R19, R2, R20, R21, R22, R23, R24, R25, R3, R4, R5, R6, R7, R8, R9: footprint Resistor_SMD:R_1206_3216Metric -> Resistor_SMD:R_1206_3216Metric_Pad1.30x1.75mm_HandSolder
Connections:
- net +3V3: now also J8.1 (Pin_1)
- net GND: now also G10.1, G9.1, J8.13 (Pin_13), J8.3 (Pin_3), J8.8 (Pin_8)
- net at U5.21 (GP16): now also J8.15 (Pin_15)
- net at U5.22 (GP17): now also J8.14 (Pin_14)
- net at U5.24 (GP18): now also J8.12 (Pin_12)
- net at U5.25 (GP19): now also J8.11 (Pin_11)
- net at U5.26 (GP20): now also J8.10 (Pin_10)
- net at U5.27 (GP21): now also J8.9 (Pin_9)
- net at U5.29 (GP22): now also J8.7 (Pin_7)
- net at U5.30 (RUN): now also J8.6 (Pin_6)
- net at U5.31 (GP26/ADC0): now also J8.5 (Pin_5)
- net at U5.32 (GP27/ADC1): now also J8.4 (Pin_4)
- net at U5.34 (GP28/ADC2): now also J8.2 (Pin_2)
- no-connect marks 16 -> 15

Commit message: Added part selection
Parts:
- C1, C15, C16, C17, C2, C24, C27, C30, C4, C5, C6: MPN (none) -> C1206C104K5RACTU
- C10, C7, C8, C9: MPN (none) -> KGM31HR71C105KU
- C11, C12, C13, C14, C26, C29: MPN (none) -> C1206C103K5RAC7210
- C18, C19, C3: MPN (none) -> C1206C106K4PACTU
- C20, C22: MPN (none) -> KGM31BCG2A181FT
- C21, C23: MPN (none) -> C3216C0G2J101G060AA
- C28, C31: MPN (none) -> ESK475M016AC3AA
- G1, G10, G2, G3, G4, G5, G6, G7, G8, G9, J6, J7, TP1, TP10, TP11, TP12, TP2, TP3, TP4, TP5, TP6, TP7, TP8: now not fitted
- J1: MPN (none) -> CONSMA001-G
- J10: Tayda (none) -> A-1069
- J2: MPN (none) -> SJ1-3515N
- J3: Adafruit PN (none) -> 2045; Tayda A-6992 -> (none)
- J4, J5: now fitted
- J8: value GPIO Breakout -> GPIO Breakout1; Tayda (none) -> A-1669
- J9: value GPIO Breakout -> GPIO Breakout2; Tayda (none) -> A-1306
- L1: MPN (none) -> LQM31PN1R5M00L
- L2, L3, L4, L5, L6: MPN (none) -> HZ1206E601R-10
- R1: MPN (none) -> CR1206-FX-62R0ELF
- R10, R11: MPN (none) -> CR1206-FX-2201ELF
- R12, R13, R14, R15, R4, R5: MPN (none) -> CR1206-FX-1002ELF
- R16, R17, R18, R19, R20, R21, R22, R23: MPN (none) -> CR1206-JW-512ELF
- R2, R3: MPN (none) -> CR1206-FX-5100ELF
- R24, R25: MPN (none) -> CRCW12060000Z0EAC
- R6, R7, R8, R9: MPN (none) -> CR1206-FX-1000ELF
- U1: MPN (none) -> GALI-S66+
- U2: MPN (none) -> SN74CBTLV3253DR
- U3, U4: MPN (none) -> MC33078DR
- U5: MPN (none) -> SC0915

Commit message: Update for Rev 2 of the board
Parts:
- added D1: 5V LED, LED_SMD:LED_1206_3216Metric_Pad1.42x1.75mm_HandSolder, symbol Device:LED
- added D2: 3V3 LED, LED_SMD:LED_1206_3216Metric_Pad1.42x1.75mm_HandSolder, symbol Device:LED
- added D3: Indicator, LED_SMD:LED_1206_3216Metric_Pad1.42x1.75mm_HandSolder, symbol Device:LED
- added R26: 3k, Resistor_SMD:R_1206_3216Metric_Pad1.30x1.75mm_HandSolder, symbol Device:R
- added R27, R28: 1k5, Resistor_SMD:R_1206_3216Metric_Pad1.30x1.75mm_HandSolder, symbol Device:R
- added TP19, TP20: TestPoint, Connector_PinHeader_2.54mm:PinHeader_1x01_P2.54mm_Vertical, symbol Connector:TestPoint
- added TPa1: LNA Bias, TestPoint:TestPoint_Pad_D1.5mm, symbol Connector:TestPoint_Probe
- added TPc1: Mixer Enable, TestPoint:TestPoint_Pad_D1.5mm, symbol Connector:TestPoint_Probe
- added TPd1: Mixer DC, TestPoint:TestPoint_Pad_D1.5mm, symbol Connector:TestPoint_Probe
- added TPe1: Q offset, TestPoint:TestPoint_Pad_D1.5mm, symbol Connector:TestPoint_Probe
- added TPf1: I offset, TestPoint:TestPoint_Pad_D1.5mm, symbol Connector:TestPoint_Probe
- added TPg1: Amp DC, TestPoint:TestPoint_Pad_D1.5mm, symbol Connector:TestPoint_Probe
- added TPh1: Filter DC, TestPoint:TestPoint_Pad_D1.5mm, symbol Connector:TestPoint_Probe
- R16, R17, R18, R19, R20, R21, R22, R23: MPN CR1206-JW-512ELF -> CR1206-FX-5101ELF
Connections:
- net +3V3: now also D2.2 (A)
- net +5V: now also D1.2 (A)
- net GND: now also J10.2 (Pin_2), R26.2, R27.2, R28.2; no longer J10.3 (Pin_3)
- net I_out: now also J10.3 (Pin_3); no longer J10.2 (Pin_2)
- net at C24.1, L4.1, U4.8 (V+): now also TPh1.1
- net at R14.2, R15.1, R7.2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: now also TPf1.1
- net at C6.2, L2.2, U2.16 (VCC): now also TPd1.1
- net at C4.1, L1.2, U1.3: now also TPa1.1
- net at C12.2, C8.1, R9.1: now also TP19.1
- net at C15.2, C16.1, C17.2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: now also TPg1.1
- net at R12.2, R13.1, R9.2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: now also TPe1.1
- net at C10.1, C14.2, R7.1: now also TP20.1
- net at R5.1, U2.1 (1~{OE}), U2.15 (2~{OE}): now also TPc1.1
- net at J8.15 (Pin_15), U5.21 (GP16): now also D3.2 (A)
- new net: D3.1 (K), R28.1
- new net: D2.1 (K), R27.1
- new net: D1.1 (K), R26.1
Other:
- note added: "Bias for 1 mA current"
- moved on the sheet: G3, L1, R1
